Commit message: target

File: config/open_manipulator_x.ros2_control.xacro (robot description, xacro)
@@ -40,5 +40,5 @@
         <state_interface name="velocity"/>
       </joint>
-      <!-- <joint name="virtual_roll_joint">
+      <joint name="virtual_roll_joint">
         <command_interface name="position"/>
         <state_interface name="position">
@@ -53,5 +53,5 @@
         </state_interface>
         <state_interface name="velocity"/>
-      </joint> -->
+      </joint>
       <joint name="gripper">
         <command_interface name="position"/>

File: urdf/open_manipulator_x.urdf.xacro (robot description, xacro)
@@ -1,12 +1,4 @@
 <?xml version="1.0"?>
 <robot name="open_manipulator_x" xmlns:xacro="http://ros.org/wiki/xacro">
-  <!-- World -->
-  <link name="world"/>
-  <!-- World fixed joint-->
-  <joint name="world_fixed" type="fixed">
-    <origin xyz="0 0 0" rpy="0 0 0"/>
-    <parent link="world"/>
-    <child link="link1"/>
-  </joint>
   <material name="grey">
     <color rgba="0.5 0.5 0.5 1.0"/>
@@ -225,8 +217,66 @@
     </inertial>
   </link>
+  <!-- Virtual roll joint -->
+  <joint name="virtual_roll_joint" type="revolute">
+    <limit lower="-3.1415" upper="3.1415" effort="54.0" velocity="3.14"/>
+    <parent link="link5"/>
+    <child link="virtual_roll_link"/>
+    <axis xyz="1 0 0"/>
+    <origin xyz="0.126 0.0 0.0" rpy="0 0 0"/>
+    <dynamics damping="0.0" friction="0.0"/>
+  </joint>
+  <!-- Virtual roll link -->
+  <link name="virtual_roll_link">
+    <visual>
+      <origin xyz="0 0 0" rpy="0 0 0"/>
+      <geometry>
+        <box size="0.01 0.01 0.01" />
+      </geometry>
+      <material name="red"/>
+     </visual>
+    <inertial>
+      <origin xyz="0 0 0" />
+      <mass value="1.0e-03" />
+      <inertia ixx="1.0e-03" ixy="0.0" ixz="0.0"
+               iyy="1.0e-03" iyz="0.0"
+               izz="1.0e-03" />
+    </inertial>
+  </link>
+  <gazebo reference="virtual_roll_link">
+    <material>Gazebo/Red</material>
+  </gazebo>
+  <!-- Virtual yaw joint -->
+  <joint name="virtual_yaw_joint" type="revolute">
+    <limit lower="-3.1415" upper="3.1415" effort="54.0" velocity="3.14"/>
+    <parent link="virtual_roll_link"/>
+    <child link="virtual_yaw_link"/>
+    <axis xyz="0 0 1"/>
+    <origin xyz="0.0 0.0 0.0" rpy="0 0 0"/>
+    <dynamics damping="0.0" friction="0.0"/>
+  </joint>
+  <!-- Virtual yaw link -->
+  <link name="virtual_yaw_link">
+    <visual>
+      <origin xyz="0 0 0" rpy="0 0 0"/>
+      <geometry>
+        <box size="0.01 0.01 0.01" />
+      </geometry>
+      <material name="red"/>
+     </visual>
+    <inertial>
+      <origin xyz="0 0 0" />
+      <mass value="1.0e-03" />
+      <inertia ixx="1.0e-03" ixy="0.0" ixz="0.0"
+               iyy="1.0e-03" iyz="0.0"
+               izz="1.0e-03" />
+    </inertial>
+  </link>
+  <gazebo reference="virtual_yaw_link">
+    <material>Gazebo/Red</material>
+  </gazebo>
   <!-- end effector joint -->
   <joint name="end_effector_joint" type="fixed">
-    <origin xyz="0.126 0.0 0.0" rpy="0 0 0"/>
-    <parent link="link5"/>
+    <origin xyz="0.0 0.0 0.0" rpy="0 0 0"/>
+    <parent link="virtual_yaw_link"/>
     <child link="end_effector_link"/>
   </joint>
